File: hardware/adapter/adapter.kicad_pcb (KiCad board)
At the start: 2 copper layers, 20.3 x 38.1 mm, 3 parts, among them J1 Conn_01x14_Pin, J2 Conn_01x14_Pin, U1 MAX2121ETI+

Commit message: fix connector
Parts:
- removed U1: MAX2121ETI+, MAX2121:21-0140L_T2855-3_MXM
- added J10: Conn_01x01_Pin, Connector_PinHeader_2.54mm:PinHeader_1x01_P2.54mm_Vertical, F.Cu at (138.2, 108.0)
- added J11: Conn_01x01_Pin, Connector_PinHeader_2.54mm:PinHeader_1x01_P2.54mm_Vertical, F.Cu at (138.2, 112.5)
- added J12: Conn_01x01_Pin, Connector_PinHeader_2.54mm:PinHeader_1x01_P2.54mm_Vertical, F.Cu at (141.9, 116.7)
- added J13: Conn_01x01_Pin, Connector_PinHeader_2.54mm:PinHeader_1x01_P2.54mm_Vertical, F.Cu at (146.7, 116.7)
- added J14: Conn_01x01_Pin, Connector_PinHeader_2.54mm:PinHeader_1x01_P2.54mm_Vertical, F.Cu at (155.7, 116.6)
- added J15: Conn_01x01_Pin, Connector_PinHeader_2.54mm:PinHeader_1x01_P2.54mm_Vertical, F.Cu at (160.3, 116.6)
- added J16: Conn_01x01_Pin, Connector_PinHeader_2.54mm:PinHeader_1x01_P2.54mm_Vertical, F.Cu at (164.2, 114.3)
- added J17: Conn_01x01_Pin, Connector_PinHeader_2.54mm:PinHeader_1x01_P2.54mm_Vertical, F.Cu at (151.2, 116.6)
- added J18: Conn_01x01_Pin, Connector_PinHeader_2.54mm:PinHeader_1x01_P2.54mm_Vertical, F.Cu at (138.3, 92.9)
- added J19: Conn_01x01_Pin, Connector_PinHeader_2.54mm:PinHeader_1x01_P2.54mm_Vertical, F.Cu at (164.2, 85.5)
- added J20: Conn_01x01_Pin, Connector_PinHeader_2.54mm:PinHeader_1x01_P2.54mm_Vertical, F.Cu at (164.1, 80.8)
- added J21: Conn_01x01_Pin, Connector_PinHeader_2.54mm:PinHeader_1x01_P2.54mm_Vertical, F.Cu at (159.8, 75.8)
- added J22: Conn_01x01_Pin, Connector_PinHeader_2.54mm:PinHeader_1x01_P2.54mm_Vertical, F.Cu at (155.6, 75.8)
- added J23: Conn_01x01_Pin, Connector_PinHeader_2.54mm:PinHeader_1x01_P2.54mm_Vertical, F.Cu at (151.2, 75.8)
- added J24: Conn_01x01_Pin, Connector_PinHeader_2.54mm:PinHeader_1x01_P2.54mm_Vertical, F.Cu at (146.8, 75.8)
- added J25: Conn_01x01_Pin, Connector_PinHeader_2.54mm:PinHeader_1x01_P2.54mm_Vertical, F.Cu at (142.4, 75.8)
- added J26: Conn_01x01_Pin, Connector_PinHeader_2.54mm:PinHeader_1x01_P2.54mm_Vertical, F.Cu at (138.2, 80.0)
- added J27: Conn_01x01_Pin, Connector_PinHeader_2.54mm:PinHeader_1x01_P2.54mm_Vertical, F.Cu at (164.2, 105.5)
- added J28: Conn_01x01_Pin, Connector_PinHeader_2.54mm:PinHeader_1x01_P2.54mm_Vertical, F.Cu at (164.2, 109.7)
- added J3: Conn_01x01_Pin, Connector_PinHeader_2.54mm:PinHeader_1x01_P2.54mm_Vertical, F.Cu at (164.2, 93.8)
- added J4: Conn_01x01_Pin, Connector_PinHeader_2.54mm:PinHeader_1x01_P2.54mm_Vertical, F.Cu at (164.2, 97.6)
- added J5: Conn_01x01_Pin, Connector_PinHeader_2.54mm:PinHeader_1x01_P2.54mm_Vertical, F.Cu at (164.2, 101.3)
- added J6: Conn_01x01_Pin, Connector_PinHeader_2.54mm:PinHeader_1x01_P2.54mm_Vertical, F.Cu at (138.2, 88.7)
- added J7: Conn_01x01_Pin, Connector_PinHeader_2.54mm:PinHeader_1x01_P2.54mm_Vertical, F.Cu at (130.9, 95.8)
- added J8: Conn_01x01_Pin, Connector_PinHeader_2.54mm:PinHeader_1x01_P2.54mm_Vertical, F.Cu at (138.3, 98.8)
- added J9: Conn_01x01_Pin, Connector_PinHeader_2.54mm:PinHeader_1x01_P2.54mm_Vertical, F.Cu at (138.3, 103.5)
- added U2: MAX2121ETI+, footprints:MAX2121ETI&plus_, F.Cu at (151.2, 95.8)
- J1, J2: value Conn_01x14_Pin -> Conn_01x01_Pin; footprint Connector_PinHeader_2.54mm:PinHeader_1x14_P2.54mm_Vertical -> Connector_PinHeader_2.54mm:PinHeader_1x01_P2.54mm_Vertical; moved to F.Cu
- moved J2 44.0 mm to (164.2, 90.1), turned to 0 degrees
- moved J1 31.8 mm to (138.2, 84.3), turned to 0 degrees
Routing:
- net Net-(J12-Pin_1): track 0.00 -> 21.9 mm
- net Net-(J15-Pin_1): track 0.00 -> 21.7 mm
- net Net-(J11-Pin_1): track 0.00 -> 21.5 mm
- net Net-(J16-Pin_1): track 0.00 -> 20.9 mm
- net Net-(J25-Pin_1): track 0.00 -> 20.9 mm
- net Net-(J21-Pin_1): track 0.00 -> 20.8 mm
- net Net-(J13-Pin_1): track 0.00 -> 20.1 mm
- net Net-(J14-Pin_1): track 0.00 -> 20.1 mm
- net Net-(J26-Pin_1): track 0.00 -> 19.4 mm
- net Net-(J24-Pin_1): track 0.00 -> 19.3 mm
- net Net-(J22-Pin_1): track 0.00 -> 19.2 mm
- net Net-(J20-Pin_1): track 0.00 -> 19.0 mm
- net Net-(J28-Pin_1): track 0.00 -> 18.5 mm
- net Net-(J17-Pin_1): track 0.00 -> 18.4 mm
- net Net-(J10-Pin_1): track 0.00 -> 18.2 mm
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Other:
- board size 20.3 x 38.1 mm -> 37.3 x 45.9 mm

Commit message: fix net
Routing:
- net Net-(J11-Pin_1): track 21.5 -> 20.4 mm
Changed lines of the file:
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@@
     (pad_to_mask_clearance 0)
     (pcbplotparams
-      (layerselection 0x00010fc_ffffffff)
-      (plot_on_all_layers_selection 0x0000000_00000000)
+      (layerselection 0x0000000_7fffffff)
+      (plot_on_all_layers_selection 0x0000000_00000001)
       (disableapertmacros false)
       (usegerberextensions false)
@@
       (sketchpadsonfab false)
       (subtractmaskfromsilk false)
-      (outputformat 1)
+      (outputformat 3)
       (mirror false)
-      (drillshape 1)
+      (drillshape 0)
       (scaleselection 1)
       (outputdirectory "")
@@
   (segment (start 145.7 100.8) (end 143 103.5) (width 0.25) (layer "F.Cu") (net 9))
   (segment (start 149.68 98.21) (end 149.68 103.37) (width 0.25) (layer "F.Cu") (net 10))
-  (segment (start 139 113.05) (end 139 111.95) (width 0.25) (layer "F.Cu") (net 10))
   (segment (start 149.68 103.37) (end 140.5 112.55) (width 0.25) (layer "F.Cu") (net 10))
   (segment (start 140.5 112.55) (end 138.25 112.55) (width 0.25) (layer "F.Cu") (net 10))
@@
   (segment (start 147.15 103.2) (end 142.3 108.05) (width 0.25) (layer "F.Cu") (net 17))
   (segment (start 148.450857 97.300857) (end 147.774383 97.325617) (width 0.25) (layer "F.Cu") (net 17))
-  (segment (start 138.68 108.887501) (end 138.762499 108.887501) (width 0.25) (layer "F.Cu") (net 17))
   (segment (start 142.3 108.05) (end 138.25 108.05) (width 0.25) (layer "F.Cu") (net 17))
   (segment (start 148.8075 97.3375) (end 148.770857 97.300857) (width 0.25) (layer "F.Cu") (net 17))
